Commit message: Changed to 4 wheels

File: urdf/aubo-i5.urdf (robot description, URDF)
Before this commit: robot aubo_i5, 21 links, 20 joints
Links:
- removed link stand_Link
Joints:
- removed joint base_to_stand_joint

File: urdf/aubo.gazebo.xacro (robot description, xacro)
@@ -7,6 +7,6 @@
 	 <!--left_wheel_Link-->
      <gazebo reference = "left_wheel_Link">
-	  <mu1 value="200.0"/>
-      <mu2 value="100.0"/>
+	  <mu1 value="2000.0"/>
+      <mu2 value="1000.0"/>
       <kp value="10000000.0" />
       <kd value="1.0" />
@@ -15,6 +15,22 @@
 	 <!--right_wheel_Link-->
      <gazebo reference = "right_wheel_Link">
-	 <mu1 value="200.0"/>
-     <mu2 value="100.0"/>
+	 <mu1 value="2000.0"/>
+     <mu2 value="1000.0"/>
+     <kp value="10000000.0" />
+     <kd value="1.0" />
+	 <material>Gazebo/Blue</material>
+     </gazebo>
+	 <!--left_wheel_Link-->
+     <gazebo reference = "left_2wheel_Link">
+	  <mu1 value="2000.0"/>
+      <mu2 value="1000.0"/>
+      <kp value="10000000.0" />
+      <kd value="1.0" />
+	  <material>Gazebo/Blue</material>
+     </gazebo>
+	 <!--right_wheel_Link-->
+     <gazebo reference = "right_2wheel_Link">
+	 <mu1 value="2000.0"/>
+     <mu2 value="1000.0"/>
      <kp value="10000000.0" />
      <kd value="1.0" />

File: urdf/aubo.transmission.xacro (robot description, xacro)
@@ -34,4 +34,22 @@
   </actuator>
   <joint name="base_to_right_wheel_joint">
+	<hardwareInterface>VelocityJointInterface</hardwareInterface>
+  </joint>
+</transmission>
+<transmission name="left_2wheel_trans">
+  <type>transmission_interface/SimpleTransmission</type>
+  <actuator name="left_2wheel_motor">
+	<mechanicalReduction>1</mechanicalReduction>
+  </actuator>
+  <joint name="base_to_left_2wheel_joint">
+	<hardwareInterface>VelocityJointInterface</hardwareInterface>
+  </joint>
+</transmission>
+<transmission name="right_2wheel_trans">
+  <type>transmission_interface/SimpleTransmission</type>
+  <actuator name="right_2wheel_motor">
+	<mechanicalReduction>1</mechanicalReduction>
+  </actuator>
+  <joint name="base_to_right_2wheel_joint">
 	<hardwareInterface>VelocityJointInterface</hardwareInterface>
   </joint>

File: urdf/aubo_i5.urdf.xacro (robot description, xacro)
@@ -3,4 +3,6 @@
 <xacro:include filename="$(find urdf_tutorial)/urdf/materials.xacro" />
 <xacro:include filename="$(find urdf_tutorial)/urdf/aubo.transmission.xacro" />
+<xacro:property name="tire_width" value="-0.06" />
+<xacro:property name="tire_radius" value="0.15" />
 <!-- MOVING_BASE_LINK -->
 <link
@@ -44,5 +46,5 @@
     <origin rpy="0 0 0" xyz="0.4 -0.275 0.42"/>
   </joint>
-<!-- LEFT WHEEL -->
+<!-- LEFT 1 WHEEL -->
 <link
     name="left_wheel_Link">
@@ -66,5 +68,5 @@
         rpy="1.571 0 0" />
       <geometry>
-        <cylinder length="0.1" radius="0.25"/>
+        <cylinder length="0.1" radius="${tire_radius}"/>
       </geometry>
       <material name="blue"/>
@@ -75,5 +77,5 @@
         rpy="0 0 0" />
       <geometry>
-	<cylinder length="0.1" radius="0.25"/>
+	<cylinder length="0.1" radius="${tire_radius}"/>
       </geometry>
     </collision>
@@ -89,35 +91,9 @@
     <parent link="moving_base_Link"/>
     <child link="left_wheel_Link"/>
-    <origin rpy="0 0 0" xyz="0.3 -0.6 0.0"/>
-  </joint>
-<!-- STAND -->
+    <origin rpy="0 0 0" xyz="0.2 -0.6 ${tire_width}"/>
+  </joint>
+<!-- LEFT 2 WHEEL -->
 <link
-    name="stand_Link">
-    <visual>
-      <origin
-        xyz="0 0 0"
-        rpy="0 0 0" />
-      <geometry>
-	<cylinder length="0.25" radius="0.02"/>
-      </geometry>
-      <material name="blue"/>
-    </visual>
-    <collision>
-      <origin
-        xyz="0 0 0"
-        rpy="0 0 0" />
-      <geometry>
-	<cylinder length="0.25" radius="0.05"/>
-      </geometry>
-    </collision>
-</link>
-  <joint name="base_to_stand_joint" type="fixed">
-    <parent link="moving_base_Link"/>
-    <child link="stand_Link"/>
-    <origin rpy="0 0 0" xyz="0.75 -0.275 -0.125"/>
-  </joint>
-<!-- RIGHT WHEEL -->
-<link
-    name="right_wheel_Link">
+    name="left_2wheel_Link">
     <inertial>
       <origin
@@ -136,8 +112,8 @@
     <visual>
       <origin
-        xyz="0 0 0"
+        xyz="0.0 0.0 0.0"
         rpy="1.571 0 0" />
       <geometry>
-	<cylinder length="0.1" radius="0.25"/>
+        <cylinder length="0.1" radius="${tire_radius}"/>
       </geometry>
       <material name="blue"/>
@@ -148,5 +124,52 @@
         rpy="0 0 0" />
       <geometry>
-	<cylinder length="0.1" radius="0.25"/>
+	<cylinder length="0.1" radius="${tire_radius}"/>
+      </geometry>
+    </collision>
+</link>
+  <joint name="base_to_left_2wheel_joint" type="continuous">
+    <axis
+      xyz="0.0 1.0 0" />
+    <limit
+      lower="-3.05"
+      upper="3.05"
+      effort="145.0"
+      velocity="3.30" />
+    <parent link="moving_base_Link"/>
+    <child link="left_2wheel_Link"/>
+    <origin rpy="0 0 0" xyz="0.6 -0.6 ${tire_width}"/>
+  </joint>
+<!-- RIGHT WHEEL -->
+<link
+    name="right_wheel_Link">
+    <inertial>
+      <origin
+        xyz="0 0 0"
+        rpy="1.571 0 0" />
+      <mass
+        value="1.5" />
+      <inertia
+        ixx="0.0164583"
+        ixy="0"
+        ixz="0"
+        iyy="0.046875"
+        iyz="0"
+        izz="0.0164583" />
+    </inertial>
+    <visual>
+      <origin
+        xyz="0 0 0"
+        rpy="1.571 0 0" />
+      <geometry>
+	<cylinder length="0.1" radius="${tire_radius}"/>
+      </geometry>
+      <material name="blue"/>
+    </visual>
+    <collision>
+      <origin
+        xyz="0 0 0"
+        rpy="0 0 0" />
+      <geometry>
+	<cylinder length="0.1" radius="${tire_radius}"/>
       </geometry>
     </collision>
@@ -162,5 +185,52 @@
     <parent link="moving_base_Link"/>
     <child link="right_wheel_Link"/>
-    <origin rpy="0 0 0" xyz="0.3 0.05 0.0"/>
+    <origin rpy="0 0 0" xyz="0.2 0.05 ${tire_width}"/>
+  </joint>
+<!-- RIGHT WHEEL 2 -->
+<link
+    name="right_2wheel_Link">
+    <inertial>
+      <origin
+        xyz="0 0 0"
+        rpy="1.571 0 0" />
+      <mass
+        value="1.5" />
+      <inertia
+        ixx="0.0164583"
+        ixy="0"
+        ixz="0"
+        iyy="0.046875"
+        iyz="0"
+        izz="0.0164583" />
+    </inertial>
+    <visual>
+      <origin
+        xyz="0 0 0"
+        rpy="1.571 0 0" />
+      <geometry>
+	<cylinder length="0.1" radius="${tire_radius}"/>
+      </geometry>
+      <material name="blue"/>
+    </visual>
+    <collision>
+      <origin
+        xyz="0 0 0"
+        rpy="0 0 0" />
+      <geometry>
+	<cylinder length="0.1" radius="${tire_radius}"/>
+      </geometry>
+    </collision>
+</link>
+  <joint name="base_to_right_2wheel_joint" type="continuous">
+    <axis
+      xyz="0 1.0 0" />
+    <limit
+      lower="-3.05"
+      upper="3.05"
+      effort="145.0"
+      velocity="3.30" />
+    <parent link="moving_base_Link"/>
+    <child link="right_2wheel_Link"/>
+    <origin rpy="0 0 0" xyz="0.6 0.05 ${tire_width}"/>
   </joint>
 <!-- BASE_LINK -->
