Commit message: Fix gripper too heavy

File: urdf/aubo_i5.urdf.xacro (robot description, xacro)
@@ -850,26 +850,4 @@
     <dynamics damping="0.0" friction="0.0"/>
   </joint>
-  <link
-     name="ee_Link">
-     <collision>
-       <geometry>
-          <box size="0.01 0.01 0.01"/>
-       </geometry>
-       <origin
-          rpy="0 0 0"
-          xyz="0 0 0.05"/>
-     </collision>
-  </link>
-  <joint
-     name="ee_fixed_joint"
-     type="fixed">
-     <parent
-	link="wrist3_Link" />
-     <child
-	link = "ee_Link" />
-     <origin
-        xyz="0.0 0.0 0.0"
-        rpy="0.0 0.0 0.0" />
-  </joint>
   <joint name="left_gripper_joint" type="revolute">
     <axis xyz="0 0 1"/>
@@ -893,6 +871,6 @@
     </collision>
     <inertial>
-      <mass value="0.05"/>
-      <inertia ixx="0.01" ixy="0.0" ixz="0.0" iyy="0.01" iyz="0.0" izz="0.01"/>
+      <mass value="0.005"/>
+      <inertia ixx="0.0001" ixy="0.0" ixz="0.0" iyy="0.0001" iyz="0.0" izz="0.0001"/>
     </inertial>
   </link>
@@ -911,6 +889,6 @@
     </collision>
     <inertial>
-      <mass value="0.05"/>
-      <inertia ixx="0.01" ixy="0.0" ixz="0.0" iyy="0.01" iyz="0.0" izz="0.01"/>
+      <mass value="0.005"/>
+      <inertia ixx="0.0001" ixy="0.0" ixz="0.0" iyy="0.0001" iyz="0.0" izz="0.0001"/>
     </inertial>
   </link>
@@ -936,6 +914,6 @@
     </collision>
     <inertial>
-      <mass value="0.05"/>
-      <inertia ixx="0.01" ixy="0.0" ixz="0.0" iyy="0.01" iyz="0.0" izz="0.01"/>
+      <mass value="0.005"/>
+      <inertia ixx="0.0001" ixy="0.0" ixz="0.0" iyy="0.0001" iyz="0.0" izz="0.0001"/>
     </inertial>
   </link>
@@ -954,6 +932,6 @@
     </collision>
     <inertial>
-      <mass value="0.05"/>
-      <inertia ixx="0.01" ixy="0.0" ixz="0.0" iyy="0.01" iyz="0.0" izz="0.01"/>
+      <mass value="0.005"/>
+      <inertia ixx="0.0001" ixy="0.0" ixz="0.0" iyy="0.0001" iyz="0.0" izz="0.0001"/>
     </inertial>
   </link>
